Commit message: i

File: description/ros2_control/diffbot.ros2_control.xacro (robot description, xacro)
@@ -5,8 +5,8 @@
       <hardware>
         <plugin>diffdrive_arduino/DiffDriveArduinoHardware</plugin>
-        <param name="rear_left_wheel_name">left_wheel_joint</param>
         <param name="front_left_wheel_name">front_left_wheel_joint</param>
-        <param name="rear_right_wheel_name">right_wheel_joint</param>
+        <param name="rear_left_wheel_name">rear_left_wheel_joint</param>
         <param name="front_right_wheel_name">front_right_wheel_joint</param>
+        <param name="rear_right_wheel_name">rear_right_wheel_joint</param>
         <param name="loop_rate">30</param>
         <param name="device">/dev/ttyUSB0</param>
@@ -19,5 +19,5 @@
         <param name="pid_o">50</param>
       </hardware>
-      <joint name="${prefix}left_wheel_joint">
+      <joint name="${prefix}rear_left_wheel_joint">
         <command_interface name="velocity"/>
         <state_interface name="position"/>
@@ -29,5 +29,5 @@
         <state_interface name="velocity"/>
       </joint>
-      <joint name="${prefix}right_wheel_joint">
+      <joint name="${prefix}reare_right_wheel_joint">
         <command_interface name="velocity"/>
         <state_interface name="position"/>

File: description/urdf/diffbot_description.urdf.xacro (robot description, xacro)
@@ -5,13 +5,17 @@
     <xacro:property name="PI" value="3.1415926535897931"/>
     <xacro:property name="base_mass" value="0.3" /> <!-- arbitrary value for base mass -->
-    <xacro:property name="base_width" value="0.2" />
-    <xacro:property name="base_length" value="0.2" />
-    <xacro:property name="base_height" value="0.05" />
+    <xacro:property name="base_width" value="0.225" />
+    <xacro:property name="base_length" value="0.153" />
+    <xacro:property name="base_height" value="0.0975" />
     <xacro:property name="wheel_mass" value="0.3" /> <!-- arbitrary value for wheel mass -->
-    <xacro:property name="wheel_len" value="0.020" />
+    <xacro:property name="wheel_len" value="0.036" />
     <xacro:property name="wheel_radius" value="0.048" />
     <xacro:property name="caster_wheel_mass" value="0.1" /> <!-- arbitrary value for caster wheel mass -->
     <xacro:property name="caster_wheel_radius" value="0.048" />
     <xacro:property name="z_offset" value="-${base_height/2}" /> <!-- Space btw top of beam and the each joint -->
+    <xacro:property name="wheel_separation" value="0.205"/>
+    <xacro:property name="wheel_offset_x" value="0.073"/>
+    <xacro:property name="wheel_offset_y" value="${wheel_separation/2}"/>
+    <xacro:property name="chassis_offset_z" value="0.02"/>
     <!-- Base Link -->
     <link name="${prefix}base_link">
@@ -23,5 +27,5 @@
       </collision>
       <visual>
-        <origin xyz="0 0 ${base_height/2}" rpy="0 0 0"/>
+        <origin xyz="0 0 ${base_height/2-chassis_offset_z}" rpy="0 0 0"/>
         <geometry>
           <box size="${base_width} ${base_length} ${base_height}"/>
@@ -29,5 +33,5 @@
         <material name="orange"/>
       </visual>
-      <inertial>
+      <!-- <inertial>
         <origin xyz="0 0 0" rpy="0 0 0"/>
         <mass value="${base_mass}"/>
@@ -36,10 +40,10 @@
           iyy="${base_mass / 12.0 * (base_height*base_height + base_width*base_width)}" iyz="0.0"
           izz="${base_mass / 12.0 * (base_width*base_width + base_length*base_length)}"/>
-      </inertial>
+      </inertial> -->
     </link>
-    <joint name="${prefix}left_wheel_joint" type="continuous">
+    <joint name="${prefix}rear_left_wheel_joint" type="continuous">
       <parent link="${prefix}base_link"/>
       <child link="${prefix}left_wheel"/>
-      <origin xyz="-0.05 -${base_width/2} ${z_offset}" rpy="0 0 0"/>
+      <origin xyz="-${wheel_offset_x} -${wheel_offset_y} 0" rpy="0 0 0"/>
       <axis xyz="0 1 0"/>
       <dynamics damping="0.2"/>
@@ -72,5 +76,5 @@
       <parent link="${prefix}base_link"/>
       <child link="${prefix}front_left_wheel"/>
-      <origin xyz="0.05 -${base_width/2} ${z_offset}" rpy="0 0 0"/>
+      <origin xyz="${wheel_offset_x} -${wheel_offset_y} 0" rpy="0 0 0"/>
       <axis xyz="0 1 0"/>
       <dynamics damping="0.2"/>
@@ -100,8 +104,8 @@
       </inertial>
     </link>
-    <joint name="${prefix}right_wheel_joint" type="continuous">
+    <joint name="${prefix}rear_right_wheel_joint" type="continuous">
       <parent link="${prefix}base_link"/>
       <child link="${prefix}right_wheel"/>
-      <origin xyz="-0.05 ${base_width/2} ${z_offset}" rpy="0 0 0"/>
+      <origin xyz="-${wheel_offset_x} ${wheel_offset_y} 0" rpy="0 0 0"/>
       <axis xyz="0 1 0"/>
       <dynamics damping="0.2"/>
@@ -134,5 +138,5 @@
       <parent link="${prefix}base_link"/>
       <child link="${prefix}front_right_wheel"/>
-      <origin xyz="0.05 ${base_width/2} ${z_offset}" rpy="0 0 0"/>
+      <origin xyz="${wheel_offset_x} ${wheel_offset_y} 0" rpy="0 0 0"/>
       <axis xyz="0 1 0"/>
       <dynamics damping="0.2"/>
@@ -162,62 +166,4 @@
       </inertial>
     </link>
-    <joint name="${prefix}caster_frontal_wheel_joint" type="fixed">
-      <parent link="${prefix}base_link"/>
-      <child link="${prefix}caster_frontal_wheel"/>
-      <origin xyz="${base_width/2 - caster_wheel_radius} 0 ${z_offset}" rpy="0 0 0"/>
-    </joint>
-    <!-- caster frontal wheel Link -->
-    <link name="${prefix}caster_frontal_wheel">
-      <collision>
-        <origin xyz="0 0 0" rpy="0 0 0"/>
-        <geometry>
-          <sphere radius="${caster_wheel_radius}"/>
-        </geometry>
-      </collision>
-      <visual>
-        <origin xyz="0 0 0" rpy="0 0 0"/>
-        <geometry>
-          <sphere radius="${caster_wheel_radius}"/>
-        </geometry>
-        <material name="white"/>
-      </visual>
-      <inertial>
-        <origin xyz="0 0 0" rpy="0 0 0"/>
-        <mass value="${caster_wheel_mass}"/>
-        <inertia
-          ixx="${caster_wheel_mass * 0.4 * (caster_wheel_radius * caster_wheel_radius)}" ixy="0.0" ixz="0.0"
-          iyy="${caster_wheel_mass * 0.4 * (caster_wheel_radius * caster_wheel_radius)}" iyz="0.0"
-          izz="${caster_wheel_mass * 0.4 * (caster_wheel_radius * caster_wheel_radius)}"/>
-      </inertial>
-    </link>
-    <joint name="${prefix}caster_rear_wheel_joint" type="fixed">
-      <parent link="${prefix}base_link"/>
-      <child link="${prefix}caster_rear_wheel"/>
-      <origin xyz="${-base_width/2 + caster_wheel_radius} 0 ${z_offset}" rpy="0 0 0"/>
-    </joint>
-    <!-- caster rear wheel Link -->
-    <link name="${prefix}caster_rear_wheel">
-      <collision>
-        <origin xyz="0 0 0" rpy="0 0 0"/>
-        <geometry>
-          <sphere radius="${caster_wheel_radius}"/>
-        </geometry>
-      </collision>
-      <visual>
-        <origin xyz="0 0 0" rpy="0 0 0"/>
-        <geometry>
-          <sphere radius="${caster_wheel_radius}"/>
-        </geometry>
-        <material name="white"/>
-      </visual>
-      <inertial>
-        <origin xyz="0 0 0" rpy="0 0 0"/>
-        <mass value="${caster_wheel_mass}"/>
-        <inertia
-          ixx="${caster_wheel_mass * 0.4 * (caster_wheel_radius * caster_wheel_radius)}" ixy="0.0" ixz="0.0"
-          iyy="${caster_wheel_mass * 0.4 * (caster_wheel_radius * caster_wheel_radius)}" iyz="0.0"
-          izz="${caster_wheel_mass * 0.4 * (caster_wheel_radius * caster_wheel_radius)}"/>
-      </inertial>
-    </link>
   </xacro:macro>
 </robot>

Commit message: i

File: description/ros2_control/diffbot.ros2_control.xacro (robot description, xacro)
@@ -29,5 +29,5 @@
         <state_interface name="velocity"/>
       </joint>
-      <joint name="${prefix}reare_right_wheel_joint">
+      <joint name="${prefix}rear_right_wheel_joint">
         <command_interface name="velocity"/>
         <state_interface name="position"/>

Commit message: i

File: description/ros2_control/diffbot.ros2_control.xacro (robot description, xacro)
@@ -10,5 +10,5 @@
         <param name="rear_right_wheel_name">rear_right_wheel_joint</param>
         <param name="loop_rate">30</param>
-        <param name="device">/dev/ttyUSB0</param>
+        <param name="device">/dev/agv-driver</param>
         <param name="baud_rate">115200</param>
         <param name="timeout_ms">1000</param>

File: description/urdf/diffbot_description.urdf.xacro (robot description, xacro)
@@ -41,4 +41,11 @@
           izz="${base_mass / 12.0 * (base_width*base_width + base_length*base_length)}"/>
       </inertial> -->
+    </link>
+    <joint name="base_footprint_joint" type="fixed">
+        <parent link="base_link"/>
+        <child link="base_footprint"/>
+        <origin xyz="0 0 -0.048" rpy="0 0 0"/>
+    </joint>
+    <link name="base_footprint">
     </link>
     <joint name="${prefix}rear_left_wheel_joint" type="continuous">
