Commit message: i

File: description/urdf/diffbot_description.urdf.xacro (robot description, xacro)
@@ -21,5 +21,5 @@
     <link name="${prefix}base_link">
       <collision>
-        <origin xyz="0 0 0" rpy="0 0 0"/>
+        <origin xyz="0 0 ${base_height/2-chassis_offset_z}" rpy="0 0 0"/>
         <geometry>
           <box size="${base_width} ${base_length} ${base_height}"/>
